Commit message: navigate action and client

File: src/robot/description/ros2_control.xacro (robot description, xacro)
@@ -5,5 +5,5 @@
         <plugin>gazebo_ros2_control/GazeboSystem</plugin>
     </hardware>
-    <joint name="left_wheel_joint">
+    <joint name="left_rear_wheel_joint">
         <command_interface name="velocity">
             <param name="min">-10</param>
@@ -13,5 +13,21 @@
         <state_interface name="velocity" />
     </joint>
-    <joint name="right_wheel_joint">
+    <joint name="right_rear_wheel_joint">
+        <command_interface name="velocity">
+            <param name="min">-10</param>
+            <param name="max">10</param>
+        </command_interface>
+        <state_interface name="position" />
+        <state_interface name="velocity" />
+    </joint>
+    <joint name="left_front_wheel_joint">
+        <command_interface name="velocity">
+            <param name="min">-10</param>
+            <param name="max">10</param>
+        </command_interface>
+        <state_interface name="position" />
+        <state_interface name="velocity" />
+    </joint>
+    <joint name="right_front_wheel_joint">
         <command_interface name="velocity">
             <param name="min">-10</param>
@@ -24,5 +40,5 @@
 <gazebo>
     <plugin filename="libgazebo_ros2_control.so" name="gazebo_ros2_control">
-        <parameters>$(find my_bot)/config/controllers.yaml </parameters>
+        <parameters>$(find robot)/config/controllers.yaml </parameters>
         <robotNamespace>/robot</robotNamespace>
     </plugin>
