Commit message: working go to waypoint controller

File: src/my_bot/description/robot.urdf.xacro (robot description, xacro)
@@ -2,4 +2,5 @@
 <robot xmlns:xacro="http://www.ros.org/wiki/xacro"  name="robot">
     <xacro:include filename="robot_core.xacro" />
-    <xacro:include filename="gazebo_control.xacro" />
+    <!-- <xacro:include filename="gazebo_control.xacro" /> -->
+    <xacro:include filename="ros2_control.xacro" />
 </robot>

File: src/my_bot/description/robot_core.xacro (robot description, xacro)
@@ -60,5 +60,5 @@
         <collision>
             <geometry>
-                <cylinder radius="0.05" length="0.04"/>
+                <sphere radius="0.05"/>
             </geometry>
         </collision>
@@ -86,5 +86,5 @@
         <collision>
             <geometry>
-                <cylinder radius="0.05" length="0.04"/>
+                <sphere radius="0.05"/>
             </geometry>
         </collision>

Commit message: nav to pose

File: src/my_bot/description/robot.urdf.xacro (robot description, xacro)
@@ -1,6 +1,25 @@
 <?xml version="1.0"?>
 <robot xmlns:xacro="http://www.ros.org/wiki/xacro"  name="robot">
+    <!-- ROVER PARAMETERS-->
+    <!-- wheel parameters -->
+    <xacro:property name="wheel_radius" value="0.05" />
+    <xacro:property name="wheel_width" value="0.05" />
+    <xacro:property name="wheel_mass" value="0.1" />
+    <!-- caster parameters -->
+    <xacro:property name="caster_radius" value="0.05" />
+    <xacro:property name="caster_position" value="0.24" />
+    <xacro:property name="caster_mass" value="0.1" />
+    <xacro:property name="caster_mu1" value="0.0001" />
+    <xacro:property name="caster_mu2" value="0.0001" />
+    <!-- chassis parameters -->
+    <xacro:property name="chassis_height" value="0.15" />
+    <xacro:property name="chassis_width" value="0.3" />
+    <xacro:property name="chassis_length" value="0.3" />
+    <xacro:property name="chassis_position" value="-0.1" />
+    <xacro:property name="chassis_mass" value="0.5" />
+    <!-- dynamic parameters -->
+    <xacro:property name="wheel_max_velocity" value="10" />
     <xacro:include filename="robot_core.xacro" />
-    <!-- <xacro:include filename="gazebo_control.xacro" /> -->
     <xacro:include filename="ros2_control.xacro" />
+    <xacro:include filename="gazebo_plugins.xacro" />
 </robot>

File: src/my_bot/description/robot_core.xacro (robot description, xacro)
@@ -21,22 +21,22 @@
         <parent link="base_link"/>
         <child link="chassis"/>
-        <origin xyz="-0.1 0 0"/>
+        <origin xyz="${chassis_position} 0 0"/>
     </joint>
     <link name="chassis">
         <visual>
-            <origin xyz="0.15 0 0.075"/>
+            <origin xyz="${chassis_length/2} 0 ${chassis_height/2}"/>
             <geometry>
-                <box size="0.3 0.3 0.15"/>
+                <box size="${chassis_length} ${chassis_width} ${chassis_height}"/>
             </geometry>
             <material name="white"/>
         </visual>
         <collision>
-            <origin xyz="0.15 0 0.075"/>
+            <origin xyz="${chassis_length/2} 0 ${chassis_height/2}"/>
             <geometry>
-                <box size="0.3 0.3 0.15"/>
+                <box size="${chassis_length} ${chassis_width} ${chassis_height}"/>
             </geometry>
         </collision>
-        <xacro:inertial_box mass="0.5" x="0.3" y="0.3" z="0.15">
-            <origin xyz="0.15 0 0.075" rpy="0 0 0"/>
+        <xacro:inertial_box mass="${chassis_mass}" x="${chassis_length}" y="${chassis_width}" z="${chassis_height}">
+            <origin xyz="${chassis_length/2} 0 ${chassis_height/2}" rpy="0 0 0"/>
         </xacro:inertial_box>
     </link>
@@ -48,5 +48,5 @@
         <parent link="base_link"/>
         <child link="left_wheel"/>
-        <origin xyz="0 0.175 0" rpy="-${pi/2} 0 0" />
+        <origin xyz="0 ${chassis_width/2 + wheel_width/2} 0" rpy="-${pi/2} 0 0" />
         <axis xyz="0 0 1"/>
     </joint>
@@ -54,5 +54,5 @@
         <visual>
             <geometry>
-                <cylinder radius="0.05" length="0.04"/>
+                <cylinder radius="${wheel_radius}" length="${wheel_width}"/>
             </geometry>
             <material name="blue"/>
@@ -60,8 +60,8 @@
         <collision>
             <geometry>
-                <sphere radius="0.05"/>
+                <sphere radius="${wheel_radius}"/>
             </geometry>
         </collision>
-        <xacro:inertial_cylinder mass="0.1" length="0.04" radius="0.05">
+        <xacro:inertial_cylinder mass="${wheel_mass}" length="${wheel_width}" radius="${wheel_radius}">
             <origin xyz="0 0 0" rpy="0 0 0"/>
         </xacro:inertial_cylinder>
@@ -74,5 +74,5 @@
         <parent link="base_link"/>
         <child link="right_wheel"/>
-        <origin xyz="0 -0.175 0" rpy="${pi/2} 0 0" />
+        <origin xyz="0 -${chassis_width/2 + wheel_width/2} 0" rpy="${pi/2} 0 0" />
         <axis xyz="0 0 -1"/>
     </joint>
@@ -80,5 +80,5 @@
         <visual>
             <geometry>
-                <cylinder radius="0.05" length="0.04"/>
+                <cylinder radius="${wheel_radius}" length="${wheel_width}"/>
             </geometry>
             <material name="blue"/>
@@ -86,8 +86,8 @@
         <collision>
             <geometry>
-                <sphere radius="0.05"/>
+                <sphere radius="${wheel_radius}"/>
             </geometry>
         </collision>
-        <xacro:inertial_cylinder mass="0.1" length="0.04" radius="0.05">
+        <xacro:inertial_cylinder mass="${wheel_mass}" length="${wheel_width}" radius="${wheel_radius}">
             <origin xyz="0 0 0" rpy="0 0 0"/>
         </xacro:inertial_cylinder>
@@ -100,10 +100,10 @@
         <parent link="chassis"/>
         <child link="caster_wheel"/>
-        <origin xyz="0.24 0 0"/>
+        <origin xyz="${caster_position} 0 0"/>
     </joint>
     <link name="caster_wheel">
         <visual>
             <geometry>
-                <sphere radius="0.05"/>
+                <sphere radius="${caster_radius}"/>
             </geometry>
             <material name="black"/>
@@ -111,8 +111,8 @@
         <collision>
             <geometry>
-                <sphere radius="0.05"/>
+                <sphere radius="${caster_radius}"/>
             </geometry>
         </collision>
-        <xacro:inertial_sphere mass="0.1" radius="0.05">
+        <xacro:inertial_sphere mass="${caster_mass}" radius="${caster_radius}">
             <origin xyz="0 0 0" rpy="0 0 0"/>
         </xacro:inertial_sphere>
@@ -120,6 +120,6 @@
     <gazebo reference="caster_wheel">
         <material>Gazebo/Black</material>
-        <mu1 value="0.001"/>
-        <mu2 value="0.001"/>
+        <mu1 value="${caster_mu1}"/>
+        <mu2 value="${caster_mu2}"/>
     </gazebo>
 </robot>

File: src/my_bot/description/ros2_control.xacro (robot description, xacro)
@@ -7,6 +7,6 @@
     <joint name="left_wheel_joint">
         <command_interface name="velocity">
-            <param name="min">-10</param>
-            <param name="max">10</param>
+            <param name="min">${-wheel_max_velocity}</param>
+            <param name="max">${wheel_max_velocity}</param>
         </command_interface>
         <state_interface name="position" />
@@ -15,6 +15,6 @@
     <joint name="right_wheel_joint">
         <command_interface name="velocity">
-            <param name="min">-10</param>
-            <param name="max">10</param>
+            <param name="min">${-wheel_max_velocity}</param>
+            <param name="max">${wheel_max_velocity}</param>
         </command_interface>
         <state_interface name="position" />
@@ -30,5 +30,4 @@
     <!-- Publish ground truth pose -->
     <plugin name="ignition::gazebo::systems::PosePublisher" filename="libignition-gazebo-pose-publisher-system.so">
-    <!-- <plugin name="gz::sim::systems::PosePublisher" filename="gz-sim-pose-publisher-system"> -->
         <!-- <publish_link_pose>true</publish_link_pose> -->
         <!-- <publish_sensor_pose>true</publish_sensor_pose> -->
